Commit message: fix(sim): URDF dimensions match real-robot RangerMiniV3Params
- wheelbase: 0.50 → 0.494 m
- track:     0.38 → 0.364 m

Per ranger_params.hpp in S-abk's jazzy fork (the real-driver source
of truth on this fork). Visual delta is <2%; the change makes the sim
kinematics directly comparable to the real-robot's CalculateSteeringAngle
and odometry integrator (which both use these constants).

File: ranger_mini_v3_description/urdf/ranger_mini_v3.xacro (robot description, xacro)
@@ -17,6 +17,6 @@
         The original RR was -0.23 / -0.206 — a typo. Fixed below.)
        ============================================================ -->
-  <xacro:property name="wheelbase_half" value="0.25"/>
-  <xacro:property name="track_half"     value="0.19"/>
+  <xacro:property name="wheelbase_half" value="0.247"/>
+  <xacro:property name="track_half"     value="0.182"/>
   <xacro:property name="steer_z"        value="-0.1"/>
   <xacro:property name="wheel_drop"     value="-0.12"/>

Commit message: feat(sim): integrate ranger_mini_v3_sim_messenger + phase 4 work into jazzy
Squash-merge of phase-4-messenger. Lands the Twist→controllers
messenger node (full real-driver interface parity), the URDF axis
fix (steering axis 0,0,1 per ROS REP-103), the dimension fix
(wheelbase 0.494, track 0.364 from RangerMiniV3Params), the /clock
QoS hardening (RELIABLE on the ros_gz_bridge), and dt instrumentation.

Phase 4 deliverable: from a /cmd_vel Twist input, the sim drives
the robot in any of four motion modes (DUAL_ACKERMAN, PARALLEL,
SPINNING, side-slip via PARALLEL) and publishes /odom, /system_state,
/motion_state, /actuator_state, /battery_state matching the real
driver's interface exactly.

Source branch retained at origin/phase-4-messenger for forensic
history of how this came together (rounds 04d through 13).

Phase rollup:
- Phase 1 (description package): squashed in earlier round
- Phase 2 (ros2_control wiring): squashed with Phase 3
- Phase 3 (Gazebo Harmonic bringup): squashed with Phase 2
- Phase 4 (Twist messenger, full state interface): THIS COMMIT

File: ranger_mini_v3_description/urdf/ranger_mini_v3.xacro (robot description, xacro)
@@ -89,7 +89,7 @@
       <parent link="base_link"/>
       <child  link="${prefix}_steering_wheel_link"/>
-      <!-- Original used axis (0,0,-1); we keep that so positive command =
-           CW seen from above, matching the real-driver kinematic model. -->
-      <axis xyz="0 0 -1"/>
+      <!-- Steering axis (0,0,1): standard ROS REP-103 convention,
+           positive joint command = CCW from above = left turn. -->
+      <axis xyz="0 0 1"/>
       <limit effort="${steer_effort}" velocity="${steer_vel}"
              lower="${-steer_limit}" upper="${steer_limit}"/>
